Commit message: Updates to arm urdf file

File: urdf/twoarm.urdf.xacro (robot description, xacro)
@@ -11,5 +11,5 @@
         <parent link="base_link"/>
         <child link="link1"/>
-        <origin xyz="0.0 0.0 0.0" rpy="0 0 0"/>
+        <origin xyz="0 0 0" rpy="0 0 0"/>
         <axis xyz="0 0 1"/>
     </joint>
@@ -41,5 +41,5 @@
         <parent link="link1"/>
         <child link="link2"/>
-        <origin xyz="${L1} 0.0 0.0" rpy="0.0 0.0 0.0"/>
+        <origin xyz="${L1} 0 0" rpy="0 0 0"/>
         <axis xyz="0 0 1"/>
     </joint>
@@ -71,5 +71,5 @@
         <parent link="link2"/>
         <child link="end_effector"/>
-        <origin xyz="${L2} 0.0 0.0" rpy="0.0 0.0 0.0"/>
+        <origin xyz="${L2} 0 0" rpy="0 0 0"/>
     </joint>
      <link name="end_effector"/>

Commit message: Added structure for arm_marker node, not working

File: urdf/twoarm.urdf.xacro (robot description, xacro)
@@ -1,9 +1,9 @@
 <robot name="i_am_arm" xmlns:xacro="http://ros.org/wiki/xacro">
-    <xacro:property name="arm_file" value="$(find homework2)/config/arm.yaml"/>
-    <xacro:property name="properties" value="${load_yaml(arm_file)}"/>
-    <xacro:property name="L1" value="${properties['Length1']}"/>
-    <xacro:property name="L2" value="${properties['Length2']}"/>
-    <xacro:property name="R1" value="${properties['Radius1']}"/>
-    <xacro:property name="R2" value="${properties['Radius2']}"/>
+    <xacro:property name="arm_yaml" value="$(find homework2)/config/arm.yaml"/>
+    <xacro:property name="arm_yaml_info" value="${load_yaml(arm_yaml)}"/>
+    <xacro:property name="L1" value="${arm_yaml_info['Length1']}"/>
+    <xacro:property name="L2" value="${arm_yaml_info['Length2']}"/>
+    <xacro:property name="R1" value="${arm_yaml_info['Radius1']}"/>
+    <xacro:property name="R2" value="${arm_yaml_info['Radius2']}"/>
     <xacro:property name="PI" value="3.141592653"/>
     <link name="base_link"/>

Commit message: Arm markers are successfully working

File: urdf/twoarm.urdf.xacro (robot description, xacro)
@@ -20,8 +20,8 @@
                 <cylinder length="${L1}" radius="${R1}"/>
             </geometry>
-            <material name="red">
-                <color rgba="1 0 0 1"/>
+            <material name="light_purple">
+                <color rgba="1 0.4 1 1"/>
             </material>
-        </visual>0
+        </visual>
         <collision>
             <origin xyz="0 0 0" rpy="0 0 0"/>
@@ -50,6 +50,6 @@
                 <cylinder length="${L2}" radius="${R2}"/>
             </geometry>
-            <material name="blue">
-                <color rgba="0 0 1 1"/>
+            <material name="dark_purple">
+                <color rgba="0.4 0.2 0.6 1"/>
             </material>
         </visual>

Commit message: Commenting and docstrings complete

File: urdf/twoarm.urdf.xacro (robot description, xacro)
@@ -8,5 +8,5 @@
     <xacro:property name="PI" value="3.141592653"/>
     <link name="base_link"/>
-    <joint name="base_joint" type="continuous">
+    <joint name="base_link1" type="continuous">
         <parent link="base_link"/>
         <child link="link1"/>
@@ -38,5 +38,5 @@
         </inertial>
     </link>
-    <joint name="link_joint" type="continuous">
+    <joint name="link1_link2" type="continuous">
         <parent link="link1"/>
         <child link="link2"/>
@@ -68,5 +68,5 @@
         </inertial>
     </link>
-    <joint name="end_joint" type="fixed">
+    <joint name="link2_endeff" type="fixed">
         <parent link="link2"/>
         <child link="end_effector"/>
